File: pcb/pcb.kicad_sch (KiCad schematic)
At the start: 0 parts

Commit message: feat: kicad files
Parts:
- added A1: SC0918, MCU:RPi_Pico_SC0918, symbol RPi_Pico:SC0918
- added BT1: Battery_Cell, symbol Device:Battery_Cell
- added C1, C2: 1u, Capacitor_THT:CP_Radial_D5.0mm_P2.50mm, symbol Device:C_Polarized
- added C3: 0.1u, Capacitor_THT:C_Disc_D5.0mm_W2.5mm_P2.50mm, symbol Device:C
- added D1: D_Schottky, Diode_THT:D_DO-35_SOD27_P10.16mm_Horizontal, symbol Device:D_Schottky
- added D2: LED, symbol Device:LED
- added MLX1: ~, Camera:MLX90640, symbol Analog:MLX90640
- added R1, R2: 2k, Resistor_THT:R_Axial_DIN0207_L6.3mm_D2.5mm_P10.16mm_Horizontal, symbol Device:R
- added R3: 330, Resistor_THT:R_Axial_DIN0207_L6.3mm_D2.5mm_P10.16mm_Horizontal, symbol Device:R
- added SST1: ~, Display:Adafruit-ST7789, symbol Display_Graphic:Adafruit-ST7789
- added U1: LD1117S33TR_SOT223, Package_TO_SOT_SMD:SOT-223-3_TabPin2, symbol Regulator_Linear:LD1117S33TR_SOT223
Connections:
- new net: BT1.1 (+), C3.1, U1.3 (VI)
- new net: A1.26 (GP20), SST1.3 (D/C)
- new net: A1.27 (GP21), SST1.4 (RST)
- new net: A1.22 (GP17), SST1.5 (~{CS})
- new net: A1.25 (GP19), SST1.6 (MOSI)
- new net: A1.24 (GP18), SST1.8 (SCK)
- new net: A1.6 (GP4), MLX1.1 (SDA), R2.2
- new net: A1.7 (GP5), MLX1.2 (SCL), R1.2
- new net: A1.39 (VSYS), D1.1 (K)
- new net: D2.1 (K), R3.1
- new net GND: A1.38 (GND), BT1.2 (-), C1.2, C2.2, C3.2, MLX1.4 (GND), R3.2, SST1.9 (GND), U1.1 (GND)
- new net VDD: C1.1, C2.1, D1.2 (A), D2.2 (A), R1.1, R2.1, SST1.11 (VIN), U1.2 (VO)
- no-connect marks 0 -> 35
Other:
- note added: "Note: For ST7789, decoupling circuitry is internal."
- company: (none) -> CU Boulder
- title: (none) -> RP2040-Based Thermal Camera

Commit message: feat: dt rather than fps
Parts:
- added TP1: ~, symbol Battery_Management:TP4056
- BT1: value Battery_Cell -> Battery
Connections:
- net GND: now also TP1.4 (OUT-); no longer BT1.2 (-)
- net VDD: now also MLX1.3 (VIN)
- net at C3.1, U1.3 (VI): now also TP1.1 (OUT+); no longer BT1.1 (+)
- new net: BT1.1 (+), TP1.2 (B+)
- new net: BT1.2 (-), TP1.3 (B-)
Other:
- note added: "MLX90640"
- note added: "ST7789"
- moved on the sheet: BT1
Changed lines of the file:
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@@
+	)
+	(junction
+		(at 217.17 109.22)
+		(diameter 0)
+		(color 0 0 0 0)
 	)
 	(junction
@@
 	)
 	(junction
+		(at 217.17 90.17)
+		(diameter 0)
+		(color 0 0 0 0)
+	)
+	(junction
 		(at 256.54 90.17)
 		(diameter 0)
@@
 	)
 	(junction
-		(at 217.17 109.22)
+		(at 69.85 78.74)
 		(diameter 0)
 		(color 0 0 0 0)
@@
 		(color 0 0 0 0)
 	)
-	(junction
-		(at 217.17 90.17)
-		(diameter 0)
-		(color 0 0 0 0)
-	)
 	(no_connect
 		(at 86.36 85.09)
@@
 	(wire
 		(pts
+			(xy 69.85 78.74) (xy 69.85 92.71)
+		)
+		(stroke
+			(width 0)
+			(type default)
+		)
+	)
+	(wire
+		(pts
 			(xy 81.28 92.71) (xy 81.28 97.79)
 		)
@@
 	(wire
 		(pts
+			(xy 194.31 100.33) (xy 194.31 106.68)
+		)
+		(stroke
+			(width 0)
+			(type default)
+		)
+	)
+	(wire
+		(pts
+			(xy 195.58 95.25) (xy 195.58 90.17)
+		)
+		(stroke
+			(width 0)
+			(type default)
+		)
+	)
+	(wire
+		(pts
+			(xy 191.77 106.68) (xy 191.77 102.87)
+		)
+		(stroke
+			(width 0)
+			(type default)
+		)
+	)
+	(wire
+		(pts
 			(xy 243.84 104.14) (xy 243.84 109.22)
 		)
@@
 	(wire
 		(pts
+			(xy 191.77 91.44) (xy 191.77 95.25)
+		)
+		(stroke
+			(width 0)
+			(type default)
+		)
+	)
+	(wire
+		(pts
 			(xy 170.18 85.09) (xy 170.18 90.17)
 		)
@@
 	(wire
 		(pts
-			(xy 204.47 109.22) (xy 217.17 109.22)
+			(xy 191.77 106.68) (xy 194.31 106.68)
 		)
 		(stroke
@@
 	(wire
 		(pts
+			(xy 195.58 90.17) (xy 217.17 90.17)
+		)
+		(stroke
+			(width 0)
+			(type default)
+		)
+	)
+	(wire
+		(pts
 			(xy 217.17 109.22) (xy 231.14 109.22)
 		)
@@
 	(wire
 		(pts
+			(xy 195.58 97.79) (xy 194.31 97.79)
+		)
+		(stroke
+			(width 0)
+			(type default)
+		)
+	)
+	(wire
+		(pts
 			(xy 39.37 90.17) (xy 39.37 78.74)
 		)
@@
 	(wire
 		(pts
+			(xy 191.77 91.44) (xy 194.31 91.44)
+		)
+		(stroke
+			(width 0)
+			(type default)
+		)
+	)
+	(wire
+		(pts
 			(xy 69.85 92.71) (xy 68.58 92.71)
 		)
@@
 	(wire
 		(pts
-			(xy 204.47 96.52) (xy 204.47 90.17)
-		)
-		(stroke
-			(width 0)
-			(type default)
-		)
-	)
-	(wire
-		(pts
 			(xy 139.7 100.33) (xy 157.48 100.33)
 		)
@@
 	(wire
 		(pts
+			(xy 195.58 102.87) (xy 195.58 109.22)
+		)
+		(stroke
+			(width 0)
+			(type default)
+		)
+	)
+	(wire
+		(pts
+			(xy 195.58 109.22) (xy 217.17 109.22)
+		)
+		(stroke
+			(width 0)
+			(type default)
+		)
+	)
+	(wire
+		(pts
 			(xy 127 50.8) (xy 69.85 50.8)
 		)
@@
 	(wire
 		(pts
+			(xy 195.58 100.33) (xy 194.31 100.33)
+		)
+		(stroke
+			(width 0)
+			(type default)
+		)
+	)
+	(wire
+		(pts
 			(xy 78.74 97.79) (xy 68.58 97.79)
 		)
@@
 	(wire
 		(pts
+			(xy 194.31 97.79) (xy 194.31 91.44)
+		)
+		(stroke
+			(width 0)
+			(type default)
+		)
+	)
+	(wire
+		(pts
 			(xy 142.24 110.49) (xy 137.16 110.49)
 		)
@@
 	(wire
 		(pts
-			(xy 204.47 104.14) (xy 204.47 109.22)
-		)
-		(stroke
-			(width 0)
-			(type default)
-		)
-	)
-	(wire
-		(pts
 			(xy 68.58 95.25) (xy 73.66 95.25)
-		)
-		(stroke
-			(width 0)
-			(type default)
-		)
-	)
-	(wire
-		(pts
-			(xy 204.47 90.17) (xy 217.17 90.17)
 		)
 		(stroke
@@
 		)
 	)
+	(text "MLX90640"
+		(exclude_from_sim no)
+		(at 55.118 94.488 0)
+		(effects
+			(font
+				(size 1.27 1.27)
+			)
+		)
+	)
 	(text "Note: For ST7789, decoupling\ncircuitry is internal."
 		(exclude_from_sim no)
 		(at 168.402 130.556 0)
+		(effects
+			(font
+				(size 1.27 1.27)
+			)
+		)
+	)
+	(text "ST7789"
+		(exclude_from_sim no)
+		(at 168.402 104.394 0)
 		(effects
 			(font
@@
 	)
 	(symbol
+		(lib_id "Battery_Management:TP4056")
+		(at 204.47 99.06 0)
+		(unit 1)
+		(exclude_from_sim no)
+		(in_bom yes)
+		(on_board yes)
+		(dnp no)
+		(property "Reference" "TP1"
+			(at 205.486 96.266 0)
+			(effects
+				(font
+					(size 1.27 1.27)
+				)
+				(justify left)
+			)
+		)
+		(property "Value" "~"
+			(at 212.09 100.33 0)
+			(effects
+				(font
+					(size 1.27 1.27)
+				)
+				(justify left)
+			)
+		)
+		(property "Footprint" ""
+			(at 204.47 99.06 0)
+			(effects
+				(font
+					(size 1.27 1.27)
+				)
+				(hide yes)
+			)
+		)
+		(property "Datasheet" ""
+			(at 204.47 99.06 0)
+			(effects
+				(font
+					(size 1.27 1.27)
+				)
+				(hide yes)
+			)
+		)
+		(property "Description" ""
+			(at 204.47 99.06 0)
+			(effects
+				(font
+					(size 1.27 1.27)
+				)
+				(hide yes)
+			)
+		)
+		(pin "2"
+		)
+		(pin "4"
+		)
+		(pin "1"
+		)
+		(pin "3"
+		)
+		(instances
+			(project ""
+				(path "/5d721aef-2807-4ff2-ba0d-6e0520bb5796"
+					(reference "TP1")
+					(unit 1)
+				)
+			)
+		)
+	)
+	(symbol
 		(lib_id "power:VDD")
 		(at 127 50.8 0)
@@
 	(symbol
 		(lib_id "Device:Battery_Cell")
-		(at 204.47 101.6 0)
+		(at 191.77 100.33 0)
 		(unit 1)
 		(exclude_from_sim no)
@@
 		(dnp no)
 		(property "Reference" "BT1"
-			(at 197.358 99.06 0)
+			(at 187.198 96.52 0)
 			(effects
 				(font
@@
 			)
 		)
-		(property "Value" "Battery_Cell"
-			(at 189.484 101.346 0)
+		(property "Value" "Battery"
+			(at 186.944 107.95 0)
 			(effects
 				(font
@@
 		)
 		(property "Footprint" ""
-			(at 204.47 100.076 90)
+			(at 191.77 98.806 90)
 			(effects
 				(font
@@
 		)
 		(property "Datasheet" "~"
-			(at 204.47 100.076 90)
+			(at 191.77 98.806 90)
 			(effects
 				(font
@@
 		)
 		(property "Description" "Single-cell battery"
-			(at 204.47 101.6 0)
-			(effects
-				(font
+			(at 191.77 100.33 0)
+			(effects
+				(font
