File: pcb/_autosave-pcb.kicad_sch (KiCad schematic)
At the start: 27 parts, among them J2 USB_C_Receptacle_PowerOnly_6P, Q1 AO3401A, U1 LD1117S33TR_SOT223, U2 MCP73831-2-OT

Commit message: feat: pcb for first tape out
Other:
- note added: "FIXME: STAT is open-drain"
Changed lines of the file:
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@@
+		)
+	)
+	(text "FIXME: STAT is open-drain"
+		(exclude_from_sim no)
+		(at 192.278 133.096 0)
+		(effects
+			(font
+				(size 1.27 1.27)
+			)
 		)
 	)
